Commit message: Stability for a few more seconds

File: src/pendulum_description/urdf/pendulum.urdf.xacro (robot description, xacro)
@@ -13,5 +13,5 @@
       <origin
         xyz="6.36331745104857E-16 -0.226629032258064 -0.5"
-        rpy="0 0 0" />
+        rpy="0 0 1.5708" />
       <mass
         value="135.625" />
@@ -268,5 +268,5 @@
     <axis
       xyz="0 0 1" />
-    <dynamics damping="0.001"/>
+    <dynamics damping="0.01"/>
   </joint>
   <link
